File: mrkeebstutorial.sch (KiCad schematic (older format))
At the start: 77 parts, among them J1 USB_B_Mini, SW1 tilde/esc, SW10 9, SW11 0, SW12 _, SW13 =/+, SW14 Backspace, SW15 M1, SW16 MXSwitch, SW17 MXSwitch, SW18 MXSwitch, SW19 MXSwitch, SW2 1, SW20 MXSwitch, SW21 MXSwitch, SW22 MXSwitch, SW23 MXSwitch, SW24 MXSwitch, SW25 MXSwitch, SW26 MXSwitch, SW27 MXSwitch, SW28 MXSwitch, SW29 MXSwitch, SW3 2, SW30 MXSwitch, SW4 3, SW5 4, SW6 5, SW7 6, SW8 7, SW9 8, U1 ATmega32U4-AU, Y1 16MHz

Commit message: fixed matrix
Parts:
- added D? (x38): 1N4148W, Diode_SMD:D_SOD-123, symbol Device:D_Small
- added SW? (x2): x, acheron_MX:MX100, symbol acheronSymbols:MXSwitch
- added SW?: c, acheron_MX:MX100, symbol acheronSymbols:MXSwitch
- added SW?: m, acheron_MX:MX100, symbol acheronSymbols:MXSwitch
- added SW?: <, acheron_MX:MX100, symbol acheronSymbols:MXSwitch
- added SW?: >, acheron_MX:MX100, symbol acheronSymbols:MXSwitch
- added SW?: Shift, acheron_MX:MX100, symbol acheronSymbols:MXSwitch
- added SW?: n, acheron_MX:MX100, symbol acheronSymbols:MXSwitch
- added SW?: b, acheron_MX:MX100, symbol acheronSymbols:MXSwitch
- added SW?: ?, acheron_MX:MX100, symbol acheronSymbols:MXSwitch
- added SW?: v, acheron_MX:MX100, symbol acheronSymbols:MXSwitch
- added SW?: M4, acheron_MX:MX100, symbol acheronSymbols:MXSwitch
- added SW?: R-shift, acheron_MX:MX100, symbol acheronSymbols:MXSwitch
- added SW?: UP, acheron_MX:MX100, symbol acheronSymbols:MXSwitch
- added SW?: LCTRL, acheron_MX:MX100, symbol acheronSymbols:MXSwitch
- added SW? (x2): Win, acheron_MX:MX100, symbol acheronSymbols:MXSwitch
- added SW? (x2): Alt, acheron_MX:MX100, symbol acheronSymbols:MXSwitch
- added SW?: Space, acheron_MX:MX100, symbol acheronSymbols:MXSwitch
- added SW?: A, acheron_MX:MX100, symbol acheronSymbols:MXSwitch
- added SW?: S, acheron_MX:MX100, symbol acheronSymbols:MXSwitch
- added SW?: D, acheron_MX:MX100, symbol acheronSymbols:MXSwitch
- added SW?: J, acheron_MX:MX100, symbol acheronSymbols:MXSwitch
- added SW?: K, acheron_MX:MX100, symbol acheronSymbols:MXSwitch
- added SW?: L, acheron_MX:MX100, symbol acheronSymbols:MXSwitch
- added SW?: M3, acheron_MX:MX100, symbol acheronSymbols:MXSwitch
- added SW?: Caps, acheron_MX:MX100, symbol acheronSymbols:MXSwitch
- added SW?: H, acheron_MX:MX100, symbol acheronSymbols:MXSwitch
- added SW?: G, acheron_MX:MX100, symbol acheronSymbols:MXSwitch
- added SW?: :, acheron_MX:MX100, symbol acheronSymbols:MXSwitch
- added SW?: F, acheron_MX:MX100, symbol acheronSymbols:MXSwitch
- added SW?: \", acheron_MX:MX100, symbol acheronSymbols:MXSwitch
- added SW?: Enter, acheron_MX:MX100, symbol acheronSymbols:MXSwitch
- added SW?: Menu, acheron_MX:MX100, symbol acheronSymbols:MXSwitch
- added SW?: DOWN, acheron_MX:MX100, symbol acheronSymbols:MXSwitch
- added SW?: RIGHT, acheron_MX:MX100, symbol acheronSymbols:MXSwitch
- added SW?: LEFT, acheron_MX:MX100, symbol acheronSymbols:MXSwitch
- SW16: value MXSwitch -> Tab
- SW17: value MXSwitch -> Q
- SW18: value MXSwitch -> W
- SW19: value MXSwitch -> E
- SW20: value MXSwitch -> R
- SW21: value MXSwitch -> T
- SW22: value MXSwitch -> Y
- SW23: value MXSwitch -> U
- SW24: value MXSwitch -> I
- SW25: value MXSwitch -> O
- SW26: value MXSwitch -> P
- SW27: value MXSwitch -> {
- SW28: value MXSwitch -> }
- SW29: value MXSwitch -> \\
- SW30: value MXSwitch -> M2
Connections:
- net labels added: Row3, Row4, Row5
- wire segments 197 -> 341
Other:
- moved on the sheet: D1, D10, D11, D12, D13, D14, D15, D16, D17, D18, D19, D2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

Commit message: fixed matrix juntions
Parts:
- SW14: value Backspace -> Backspace_200
- SW16: value Tab -> Tab_150
- SW?: value Shift -> LShift_225
- SW?: value R-shift -> R-shift_175
- SW?: value Enter -> Enter_2.25
Connections:
- net Col1: no longer D1.1 (K), D10.1 (K), D11.1 (K), D12.1 (K), D13.1 (K), D14.1 (K), D15.1 (K), D16.1 (K), D17.1 (K), D18.1 (K), D19.1 (K), D2.1 (K), D20.1 (K), D21.1 (K), D22.1 (K), D23.1 (K), D24.1 (K), D25.1 (K), D26.1 (K), D27.1 (K), D28.1 (K), D29.1 (K), D3.1 (K), D30.1 (K), D4.1 (K), D5.1 (K), D6.1 (K), D7.1 (K), D8.1 (K), D9.1 (K), D?.1 (K), D?.1 (K), D?.1 (K), D?.1 (K), D?.1 (K), D?.1 (K), D?.1 (K), D?.1 (K), D?.1 (K), D?.1 (K), D?.1 (K), D?.1 (K), D?.1 (K), D?.1 (K), SW10.1 (Col), SW11.1 (Col), SW12.1 (Col), SW13.1 (Col), SW14.1 (Col), SW15.1 (Col), SW17.1 (Col), SW18.1 (Col), SW19.1 (Col), SW2.1 (Col), SW20.1 (Col), SW21.1 (Col), SW22.1 (Col), SW23.1 (Col), SW24.1 (Col), SW25.1 (Col), SW26.1 (Col), SW27.1 (Col), SW28.1 (Col), SW29.1 (Col), SW3.1 (Col), SW30.1 (Col), SW4.1 (Col), SW5.1 (Col), SW6.1 (Col), SW7.1 (Col), SW8.1 (Col), SW9.1 (Col), SW?.1 (Col), SW?.1 (Col), SW?.1 (Col), SW?.1 (Col), SW?.1 (Col), SW?.1 (Col), SW?.1 (Col), SW?.1 (Col), SW?.1 (Col), SW?.1 (Col), SW?.1 (Col), SW?.1 (Col), SW?.1 (Col), SW?.1 (Col), SW?.1 (Col), SW?.1 (Col), SW?.1 (Col), SW?.1 (Col), SW?.1 (Col), SW?.1 (Col), SW?.1 (Col), SW?.1 (Col), SW?.1 (Col), SW?.1 (Col), SW?.1 (Col), SW?.1 (Col), SW?.1 (Col), SW?.1 (Col), SW?.1 (Col), SW?.1 (Col), SW?.1 (Col), SW?.1 (Col), SW?.1 (Col), SW?.1 (Col), SW?.1 (Col)
- new net Col10: SW10.1 (Col), SW25.1 (Col), SW?.1 (Col), SW?.1 (Col), SW?.1 (Col)
- new net Col11: SW11.1 (Col), SW26.1 (Col), SW?.1 (Col), SW?.1 (Col), SW?.1 (Col)
- new net Col12: SW12.1 (Col), SW27.1 (Col), SW?.1 (Col), SW?.1 (Col), SW?.1 (Col)
- new net Col13: SW13.1 (Col), SW28.1 (Col), SW?.1 (Col), SW?.1 (Col)
- new net Col14: SW14.1 (Col), SW29.1 (Col), SW?.1 (Col), SW?.1 (Col), SW?.1 (Col)
- new net Col15: D?.1 (K), D?.1 (K), D?.1 (K), D?.1 (K), D?.1 (K), D?.1 (K), D?.1 (K), D?.1 (K), D?.1 (K), D?.1 (K), D?.1 (K), D?.1 (K), D?.1 (K), D?.1 (K), SW15.1 (Col), SW30.1 (Col), SW?.1 (Col), SW?.1 (Col), SW?.1 (Col)
- new net Col2: SW17.1 (Col), SW2.1 (Col), SW?.1 (Col), SW?.1 (Col)
- new net Col3: SW18.1 (Col), SW3.1 (Col), SW?.1 (Col), SW?.1 (Col), SW?.1 (Col)
- new net Col4: SW19.1 (Col), SW4.1 (Col), SW?.1 (Col), SW?.1 (Col)
- new net Col5: SW20.1 (Col), SW5.1 (Col), SW?.1 (Col), SW?.1 (Col)
- new net Col6: SW21.1 (Col), SW6.1 (Col), SW?.1 (Col), SW?.1 (Col)
- new net Col7: SW22.1 (Col), SW7.1 (Col), SW?.1 (Col), SW?.1 (Col), SW?.1 (Col)
- new net Col8: SW23.1 (Col), SW8.1 (Col), SW?.1 (Col), SW?.1 (Col)
- new net Col9: SW24.1 (Col), SW9.1 (Col), SW?.1 (Col), SW?.1 (Col)
- new net Row1: D1.1 (K), D10.1 (K), D11.1 (K), D12.1 (K), D13.1 (K), D14.1 (K), D15.1 (K), D2.1 (K), D3.1 (K), D4.1 (K), D5.1 (K), D6.1 (K), D7.1 (K), D8.1 (K), D9.1 (K)
- new net Row2: D16.1 (K), D17.1 (K), D18.1 (K), D19.1 (K), D20.1 (K), D21.1 (K), D22.1 (K), D23.1 (K), D24.1 (K), D25.1 (K), D26.1 (K), D27.1 (K), D28.1 (K), D29.1 (K), D30.1 (K)
Changed lines of the file:
@@
 	3825 2400 3825 2300
 Wire Wire Line
-	3825 2300 3300 2300
-Connection ~ 3300 2300
-Wire Wire Line
 	3475 2950 3300 2950
-Wire Wire Line
-	3300 2950 3300 2300
-Wire Wire Line
-	3300 2300 3300 1975
-Wire Wire Line
-	3300 2300 2900 2300
 Text GLabel 3300 1975 1    50   Input ~ 0
 Col2
@@
 	4750 2400 4750 2300
 Wire Wire Line
-	4750 2300 4225 2300
-Connection ~ 4225 2300
-Wire Wire Line
 	4400 2950 4225 2950
-Wire Wire Line
-	4225 2950 4225 2300
-Wire Wire Line
-	4225 2300 4225 1975
-Wire Wire Line
-	4225 2300 3825 2300
 Text GLabel 4225 1975 1    50   Input ~ 0
 Col3
@@
 	5675 2400 5675 2300
 Wire Wire Line
-	5675 2300 5150 2300
-Connection ~ 5150 2300
-Wire Wire Line
 	5325 2950 5150 2950
-Wire Wire Line
-	5150 2950 5150 2300
-Wire Wire Line
-	5150 2300 5150 1975
-Wire Wire Line
-	5150 2300 4750 2300
 Text GLabel 5150 1975 1    50   Input ~ 0
 Col4
@@
 	6600 2400 6600 2300
 Wire Wire Line
-	6600 2300 6075 2300
-Connection ~ 6075 2300
-Wire Wire Line
 	6250 2950 6075 2950
-Wire Wire Line
-	6075 2950 6075 2300
-Wire Wire Line
-	6075 2300 6075 1975
-Wire Wire Line
-	6075 2300 5675 2300
 Text GLabel 6075 1975 1    50   Input ~ 0
 Col5
@@
 	7525 2400 7525 2300
 Wire Wire Line
-	7525 2300 7000 2300
-Connection ~ 7000 2300
-Wire Wire Line
 	7175 2950 7000 2950
-Wire Wire Line
-	7000 2950 7000 2300
-Wire Wire Line
-	7000 2300 7000 1975
-Wire Wire Line
-	7000 2300 6600 2300
 Text GLabel 7000 1975 1    50   Input ~ 0
 Col6
@@
 Wire Wire Line
 	8450 2400 8450 2300
-Connection ~ 7925 2300
 Wire Wire Line
 	8100 2950 7925 2950
-Wire Wire Line
-	7925 2950 7925 2300
-Wire Wire Line
-	7925 2300 7525 2300
 Text GLabel 7925 1975 1    50   Input ~ 0
 Col7
@@
 $EndComp
 Wire Wire Line
-	8850 2025 8850 2300
-Connection ~ 9775 2300
-Wire Wire Line
 	9950 2950 9775 2950
-Wire Wire Line
-	9775 2950 9775 2300
-Wire Wire Line
-	9775 2300 9775 1975
 $Comp
 L acheronSymbols:MXSwitch SW8
@@
 Col8
 Wire Wire Line
-	7925 2300 7925 1975
-Wire Wire Line
-	8450 2300 7925 2300
-Wire Wire Line
-	8850 2300 8450 2300
-Connection ~ 8850 2300
-Wire Wire Line
 	9375 2400 9375 2300
-Wire Wire Line
-	9375 2300 9775 2300
 $Comp
 L Device:D_Small D9
@@
 Wire Wire Line
 	10300 2400 10300 2300
-Wire Wire Line
-	10300 2300 9775 2300
 $Comp
 L Device:D_Small D10
@@
 	11225 2400 11225 2300
 Wire Wire Line
-	11225 2300 10700 2300
-Connection ~ 10700 2300
-Wire Wire Line
 	10875 2950 10700 2950
-Wire Wire Line
-	10700 2950 10700 2300
-Wire Wire Line
-	10700 2300 10700 1975
-Wire Wire Line
-	10700 2300 10300 2300
 $Comp
 L acheronSymbols:MXSwitch SW11
@@
 	12150 2400 12150 2300
 Wire Wire Line
-	12150 2300 11625 2300
-Connection ~ 11625 2300
-Wire Wire Line
 	11800 2950 11625 2950
-Wire Wire Line
-	11625 2950 11625 2300
-Wire Wire Line
-	11625 2300 11625 1975
-Wire Wire Line
-	11625 2300 11225 2300
 $Comp
 L acheronSymbols:MXSwitch SW12
@@
 	13075 2400 13075 2300
 Wire Wire Line
-	13075 2300 12550 2300
-Connection ~ 12550 2300
-Wire Wire Line
 	12725 2950 12550 2950
-Wire Wire Line
-	12550 2950 12550 2300
-Wire Wire Line
-	12550 2300 12550 1975
-Wire Wire Line
-	12550 2300 12150 2300
 $Comp
 L acheronSymbols:MXSwitch SW13
@@
 	14000 2400 14000 2300
 Wire Wire Line
-	14000 2300 13475 2300
-Connection ~ 13475 2300
-Wire Wire Line
 	13650 2950 13475 2950
-Wire Wire Line
-	13475 2950 13475 2300
-Wire Wire Line
-	13475 2300 13475 1975
-Wire Wire Line
-	13475 2300 13075 2300
 $Comp
 L acheronSymbols:MXSwitch SW14
@@
 P 14925 2950
 F 0 "SW14" H 14850 2975 50  0000 L CNN
-F 1 "Backspace" H 14775 2875 39  0000 L CNN
+F 1 "Backspace_200" H 14725 2875 39  0000 L CNN
 F 2 "acheron_MX:MX100" H 14925 2950 50  0001 C CNN
 F 3 "" H 14925 2950 50  0001 C CNN
@@
 Wire Wire Line
 	14925 2400 14925 2300
-Connection ~ 14400 2300
-Wire Wire Line
-	14400 2950 14400 2300
-Wire Wire Line
-	14400 2300 14400 1975
-Wire Wire Line
-	14400 2300 14000 2300
 $Comp
 L acheronSymbols:MXSwitch SW15
@@
 Wire Wire Line
 	15825 2400 15825 2300
-Wire Wire Line
-	15825 2300 15300 2300
-Connection ~ 15300 2300
-Wire Wire Line
-	15300 2950 15300 2300
-Wire Wire Line
-	15300 2300 15300 1975
-Wire Wire Line
-	14400 2300 14925 2300
 Connection ~ 10300 2300
 Connection ~ 11225 2300
 Connection ~ 12150 2300
-Connection ~ 13075 2300
 Connection ~ 14000 2300
 Connection ~ 14925 2300
-Wire Wire Line
-	14925 2300 15300 2300
 $Comp
 L acheronSymbols:MXSwitch SW10
@@
 Text GLabel 15300 1975 1    50   Input ~ 0
 Col15
-Wire Wire Line
-	9375 2300 8850 2300
 Connection ~ 9375 2300
 Wire Wire Line
@@
 	2900 3400 2900 3325
 Wire Wire Line
-	2900 3325 2500 3325
-Wire Wire Line
 	2550 3950 2500 3950
-Wire Wire Line
-	2500 3950 2500 3325
-Connection ~ 2500 3325
-Wire Wire Line
-	2500 3325 2500 2950
-Wire Wire Line
-	2500 3325 1875 3325
 Text GLabel 1875 3325 0    50   Input ~ 0
 Row2
@@
 Connection ~ 14925 3325
 $Comp
-L acheronSymbols:MXSwitch SW16
-U 1 1 5F425366
-P 2900 3950
-F 0 "SW16" H 2825 3975 50  0000 L CNN
-F 1 "Tab" H 2850 3875 39  0000 L CNN
-F 2 "acheron_MX:MX100" H 2900 3950 50  0001 C CNN
-F 3 "" H 2900 3950 50  0001 C CNN
-	1    2900 3950
-	1    0    0    -1
-$EndComp
-$Comp
 L acheronSymbols:MXSwitch SW22
 U 1 1 5F4253DD
@@
 	2900 4400 2900 4325
 Wire Wire Line
-	2900 4325 2500 4325
-Wire Wire Line
 	2550 4950 2500 4950
-Connection ~ 2500 4325
-Wire Wire Line
-	2500 4325 2500 3950
-Wire Wire Line
-	2500 4325 1875 4325
 Text GLabel 1875 4325 0    50   Input ~ 0
 Row3
@@
 Wire Wire Line
 	5150 4950 5150 3950
-Wire Wire Line
-	2500 4950 2500 4325
 Wire Wire Line
 	2900 5400 2900 5325
@@
 Wire Wire Line
 	8450 3325 9375 3325
-Wire Wire Line
-	8850 2300 8850 2950
 Connection ~ 8850 2950
 Wire Wire Line
@@
 Connection ~ 3300 4950
 Connection ~ 3300 3950
-Connection ~ 3300 2950
 Connection ~ 4225 2950
 Connection ~ 4225 3950
@@
 P 14000 5950
 F 0 "SW?" H 13925 5975 50  0000 L CNN
-F 1 "R-shift" H 13900 5875 39  0000 L CNN
+F 1 "R-shift_175" H 13825 5900 39  0000 L CNN
 F 2 "acheron_MX:MX100" H 14000 5950 50  0001 C CNN
 F 3 "" H 14000 5950 50  0001 C CNN
@@
 P 14925 4950
 F 0 "SW?" H 14850 4975 50  0000 L CNN
-F 1 "Enter" H 14850 4875 39  0000 L CNN
+F 1 "Enter_2.25" H 14775 4875 39  0000 L CNN
 F 2 "acheron_MX:MX100" H 14925 4950 50  0001 C CNN
 F 3 "" H 14925 4950 50  0001 C CNN
@@
 P 2900 5950
 F 0 "SW?" H 2825 5975 50  0000 L CNN
-F 1 "Shift" H 2775 5875 79  0000 L CNN
+F 1 "LShift_225" H 2600 5850 79  0000 L CNN
 F 2 "acheron_MX:MX100" H 2900 5950 50  0001 C CNN
 F 3 "" H 2900 5950 50  0001 C CNN
@@
 Row5
 Connection ~ 13475 5950
+$Comp
+L acheronSymbols:MXSwitch SW16
+U 1 1 5F425366
+P 2900 3950
+F 0 "SW16" H 2825 3975 50  0000 L CNN
+F 1 "Tab_150" H 2800 3875 39  0000 L CNN
+F 2 "acheron_MX:MX100" H 2900 3950 50  0001 C CNN
+F 3 "" H 2900 3950 50  0001 C CNN
+	1    2900 3950
+	1    0    0    -1
+$EndComp
+Wire Wire Line
+	14400 1975 14400 2950
+Wire Wire Line
+	14000 2300 14925 2300
+Wire Wire Line
+	13075 2300 14000 2300
+Wire Wire Line
+	13475 1975 13475 2950
+Connection ~ 13075 2300
+Wire Wire Line
+	12550 1975 12550 2950
+Wire Wire Line
+	12150 2300 13075 2300
+Wire Wire Line
+	11225 2300 12150 2300
+Wire Wire Line
+	11625 1975 11625 2950
+Wire Wire Line
+	14925 2300 15825 2300
+Wire Wire Line
+	15300 1975 15300 2950
+Wire Wire Line
+	10300 2300 11225 2300
+Wire Wire Line
+	10700 1975 10700 2950
+Wire Wire Line
+	9775 1975 9775 2950
+Wire Wire Line
+	9375 2300 10300 2300
+Wire Wire Line
+	8850 2025 8850 2950
+Wire Wire Line
+	8450 2300 9375 2300
+Wire Wire Line
+	7925 1975 7925 2950
+Wire Wire Line
+	7525 2300 8450 2300
+Wire Wire Line
+	6600 2300 7525 2300
+Wire Wire Line
+	7000 1975 7000 2950
+Wire Wire Line
+	5675 2300 6600 2300
+Wire Wire Line
+	6075 1975 6075 2950
+Wire Wire Line
+	4750 2300 5675 2300
+Wire Wire Line
+	5150 1975 5150 2950
+Wire Wire Line
+	3825 2300 4750 2300
+Wire Wire Line
+	4225 1975 4225 2950
+Connection ~ 3300 2950
+Wire Wire Line
+	2900 2300 3825 2300
+Wire Wire Line
+	3300 1975 3300 2950
+Wire Wire Line
+	1875 3325 2900 3325
+Wire Wire Line
+	2500 2950 2500 3950
+Wire Wire Line
+	1875 4325 2900 4325
+Wire Wire Line
+	2500 3950 2500 4950
 $EndSCHEMATC

Commit message: semi finished scematic
Parts:
- SW14: footprint acheron_MX:MX100 -> acheron_MX:MX200
- SW16: footprint acheron_MX:MX100 -> acheron_MX:MX150
- SW31, SW56: renamed from SW?; footprint acheron_MX:MX100 -> acheron_MX:MX175
- SW43, SW45: renamed from SW?; footprint acheron_MX:MX100 -> acheron_MX:MX225
- SW59, SW60, SW61: renamed from SW?; footprint acheron_MX:MX100 -> acheron_MX:MX125
- SW62: renamed from SW?; footprint acheron_MX:MX100 -> acheron_MX:MX625R
- gave numbers to parts that had none: 68
- renumbered C5 to C1, C6 to C2, C7 to C3, C8 to C4, C1 to C5, C2 to C6, C3 to C7, C4 to C8, R2 to R1, R1 to R2

Commit message: grind done
Parts:
- SW29: footprint acheron_MX:MX100 -> acheron_MX:MX150
- SW46: value x -> z
Changed lines of the file:
@@
 F 0 "SW29" H 14850 3975 50  0000 L CNN
 F 1 "\\" H 14950 3850 39  0000 L CNN
-F 2 "acheron_MX:MX100" H 14925 3950 50  0001 C CNN
+F 2 "acheron_MX:MX150" H 14925 3950 50  0001 C CNN
 F 3 "" H 14925 3950 50  0001 C CNN
 	1    14925 3950
@@
 P 4750 5950
 F 0 "SW46" H 4675 5975 50  0000 L CNN
-F 1 "x" H 4725 5875 39  0000 L CNN
+F 1 "z" H 4725 5875 39  0000 L CNN
 F 2 "acheron_MX:MX100" H 4750 5950 50  0001 C CNN
 F 3 "" H 4750 5950 50  0001 C CNN

Commit message: pp
Parts:
- R2: value 10k -> 330
Connections:
- net GND: now also C5.1
- net at R2.2, SWP1.1: no longer C5.1
Other:
- moved on the sheet: R1, R2
Changed lines of the file:
@@
 Col1
 Wire Wire Line
-	-3275 400  -3275 325
-Wire Wire Line
-	-3275 125  -3150 125
-Connection ~ -3275 125
+	-3400 475  -3400 400
 Wire Wire Line
 	-3150 125  -3150 -100
-Wire Wire Line
-	-3400 125  -3275 125
 $Comp
 L Device:R_Small R2
 U 1 1 5F0D206C
-P -3275 225
-F 0 "R2" H -3216 271 50  0000 L CNN
-F 1 "10k" H -3216 180 50  0000 L CNN
-F 2 "Resistor_SMD:R_1206_3216Metric_Pad1.42x1.75mm_HandSolder" H -3275 225 50  0001 C CNN
-F 3 "~" H -3275 225 50  0001 C CNN
-	1    -3275 225
+P -3400 300
+F 0 "R2" H -3341 346 50  0000 L CNN
+F 1 "330" H -3341 255 50  0000 L CNN
+F 2 "Resistor_SMD:R_1206_3216Metric_Pad1.42x1.75mm_HandSolder" H -3400 300 50  0001 C CNN
+F 3 "~" H -3400 300 50  0001 C CNN
+	1    -3400 300
 	-1   0    0    1
 $EndComp
@@
 L Device:R_Small R1
 U 1 1 5F0AD905
-P -3150 -425
-F 0 "R1" H -3091 -379 50  0000 L CNN
-F 1 "10k" H -3091 -470 50  0000 L CNN
-F 2 "Resistor_SMD:R_1206_3216Metric_Pad1.42x1.75mm_HandSolder" H -3150 -425 50  0001 C CNN
-F 3 "~" H -3150 -425 50  0001 C CNN
-	1    -3150 -425
-	1    0    0    -1
-$EndComp
-Wire Wire Line
-	-3400 -300 -3150 -300
+P -3300 -400
+F 0 "R1" H -3225 -300 50  0000 L CNN
+F 1 "10k" H -3250 -400 50  0000 L CNN
+F 2 "Resistor_SMD:R_1206_3216Metric_Pad1.42x1.75mm_HandSolder" H -3300 -400 50  0001 C CNN
+F 3 "~" H -3300 -400 50  0001 C CNN
+	1    -3300 -400
+	1    0    0    -1
+$EndComp
+Wire Wire Line
+	-3400 -300 -3300 -300
 Wire Wire Line
 	-3400 -275 -3400 -300
@@
 U 1 1 5F0AD91B
 P -3400 -75
-F 0 "SWP1" V -3375 225 50  0000 R CNN
-F 1 "SW_Push" V -3475 325 50  0000 R CNN
+F 0 "SWP1" H -3300 175 50  0000 R CNN
+F 1 "SW_Push" H -3200 100 50  0000 R CNN
 F 2 "random-keyboard-parts:SKQG-1155865" H -3400 125 50  0001 C CNN
 F 3 "~" H -3400 125 50  0001 C CNN
@@
 	-3150 -300 -3000 -300
 Connection ~ -3150 -300
-Wire Wire Line
-	-3150 -325 -3150 -300
 $Comp
 L Device:C_Small C5
@@
 $EndComp
 Wire Wire Line
-	-3150 -600 -3150 -525
+	-3300 -575 -3300 -500
 $Comp
 L power:GND #PWR04
 U 1 1 5F0AD90D
-P -3275 400
-F 0 "#PWR04" H -3275 150 50  0001 C CNN
-F 1 "GND" H -3270 227 50  0000 C CNN
-F 2 "" H -3275 400 50  0001 C CNN
-F 3 "" H -3275 400 50  0001 C CNN
-	1    -3275 400
+P -3400 475
+F 0 "#PWR04" H -3400 225 50  0001 C CNN
+F 1 "GND" H -3395 302 50  0000 C CNN
+F 2 "" H -3400 475 50  0001 C CNN
+F 3 "" H -3400 475 50  0001 C CNN
+	1    -3400 475
 	1    0    0    -1
 $EndComp
@@
 L power:+5V #PWR02
 U 1 1 5F0AD8FF
-P -3150 -600
-F 0 "#PWR02" H -3150 -750 50  0001 C CNN
-F 1 "+5V" H -3135 -427 50  0000 C CNN
-F 2 "" H -3150 -600 50  0001 C CNN
-F 3 "" H -3150 -600 50  0001 C CNN
-	1    -3150 -600
+P -3300 -575
+F 0 "#PWR02" H -3300 -725 50  0001 C CNN
+F 1 "+5V" H -3285 -402 50  0000 C CNN
+F 2 "" H -3300 -575 50  0001 C CNN
+F 3 "" H -3300 -575 50  0001 C CNN
+	1    -3300 -575
 	1    0    0    -1
 $EndComp
@@
 Wire Wire Line
 	2500 3950 2500 4950
+$Comp
+L power:GND #PWR?
+U 1 1 5F0E6A56
+P -3150 125
+F 0 "#PWR?" H -3150 -125 50  0001 C CNN
+F 1 "GND" H -3145 -48 50  0000 C CNN
+F 2 "" H -3150 125 50  0001 C CNN
+F 3 "" H -3150 125 50  0001 C CNN
+	1    -3150 125
+	1    0    0    -1
+$EndComp
+Wire Wire Line
+	-3400 125  -3400 200
+Connection ~ -3300 -300
+Wire Wire Line
+	-3300 -300 -3150 -300
 $EndSCHEMATC

Commit message: connecto
Parts:
- D1, D10, D11, D12, D13, D14, D15, D16, D17, D18, D19, D2, D20, D21, D22, D23, D24, D25, D26, D27, D28, D29, D3, D30, D31, D32, D33, D34, D35, D36, D37, D38, D39, D4, D40, D41, D42, D43, D44, D45, D46, D47, D48, D49, D5, D50, D51, D52, D53, D54, D55, D56, D57, D58, D59, D6, D60, D61, D62, D63, D64, D65, D66, D67, D68, D7, D8, D9: footprint Diode_SMD:D_SOD-123 -> acheron_Components:D_THT_7.62mm_SOD-123
Connections:
- net Col1: now also U1.8 (PB0)
- net Col10: now also U1.32 (PC7)
- net Col11: now also U1.18 (PD0)
- net Col12: now also U1.19 (PD1)
- net Col13: now also U1.20 (PD2)
- net Col14: now also U1.21 (PD3)
- net Col15: now also U1.25 (PD4), U1.27 (PD7)
- net Col2: now also U1.9 (PB1)
- net Col3: now also U1.10 (PB2)
- net Col4: now also U1.11 (PB3)
- net Col5: now also U1.28 (PB4)
- net Col6: now also U1.29 (PB5)
- net Col7: now also U1.30 (PB6)
- net Col8: now also U1.12 (PB7)
- net Col9: now also U1.31 (PC6)
- net Row1: now also U1.22 (PD5)
- net Row2: now also U1.26 (PD6)
- net Row5: now also D66.1 (K)
