File: mrkeebstutorial.sch (KiCad schematic (older format))
At the start: 154 parts, among them J1 USB_B_Mini, SW1 tilde/esc, SW10 9, SW11 0, SW12 _, SW13 =/+, SW14 Backspace_200, SW15 M1, SW16 Tab_150, SW17 Q, SW18 W, SW19 E, SW2 1, SW20 R, SW21 T, SW22 Y, SW23 U, SW24 I, SW25 O, SW26 P, SW27 {, SW28 }, SW29 \\, SW3 2, SW30 M2, SW31 Caps, SW32 A, SW33 S, SW34 D, SW35 F, SW36 G, SW37 H, SW38 J, SW39 K, SW4 3, SW40 L, SW41 :, SW42 \", SW43 Enter_2.25, SW44 M3, SW45 LShift_225, SW46 z, SW47 x, SW48 c, SW49 v, SW5 4, SW50 b, SW51 n, SW52 m, SW53 <, SW54 >, SW55 ?, SW56 R-shift_175, SW57 UP, SW58 M4, SW59 LCTRL, SW6 5, SW60 Win, SW61 Alt, SW62 Space, SW63 Alt, SW64 Win, SW65 Menu, SW66 LEFT, SW67 DOWN, SW68 RIGHT, SW7 6, SW8 7, SW9 8, U1 ATmega32U4-AU, Y1 16MHz

Commit message: finare
Parts:
- removed C9: 100n, Capacitor_SMD:C_0805_2012Metric_Pad1.15x1.40mm_HandSolder, symbol Device:C_Small
- C1: LCSC C15850 -> C17024
- C3, C4, C5: LCSC C49678 -> C129690
- C6, C7: LCSC C1804 -> C465168
- D1, D10, D11, D12, D13, D14, D15, D16, D17, D18, D19, D2, D20, D21, D22, D23, D24, D25, D26, D27, D28, D29, D3, D30, D31, D32, D33, D34, D35, D36, D37, D38, D39, D4, D40, D41, D42, D43, D44, D45, D46, D47, D48, D49, D5, D50, D51, D52, D53, D54, D55, D56, D57, D58, D59, D6, D60, D61, D62, D63, D64, D65, D66, D67, D68, D7, D8, D9: LCSC C444720 -> C2099
- R1: LCSC C17414 -> C103904
- R2: LCSC C17630 -> C25306
- R3, R4: LCSC C17561 -> C17513
- R5: LCSC C17513 -> C510146
- SWP1: LCSC C318884 -> C202387
- U1: LCSC C44854 -> C44854
- Y1: LCSC C112572 -> C341521
Connections:
- net GND: no longer J1.5 (GND)
