File: mrkeebstutorial.kicad_pcb (KiCad board)
At the start: 2 copper layers, 25 parts, among them J1 USB_B_Mini, SW2 MXSwitch, SW3 MXSwitch, SW4 MXSwitch, SW5 MXSwitch, U1 ATmega32U4-AU, Y1 16MHz

Commit message: some shit was doned
Parts:
- added D10: 1N4148W, Diode_SMD:D_SOD-123, F.Cu at (5.62, -315.7)
- added D11: 1N4148W, Diode_SMD:D_SOD-123, B.Cu at (120.0, -181.1)
- added D12: 1N4148W, Diode_SMD:D_SOD-123, B.Cu at (35.5, -263.6)
- added D13: 1N4148W, Diode_SMD:D_SOD-123, B.Cu at (29.8, -267.0)
- added D14: 1N4148W, Diode_SMD:D_SOD-123, B.Cu at (114.2, -184.5)
- added D15: 1N4148W, Diode_SMD:D_SOD-123, B.Cu at (35.5, -267.0)
- added D16: 1N4148W, Diode_SMD:D_SOD-123, B.Cu at (120.0, -184.5)
- added D17: 1N4148W, Diode_SMD:D_SOD-123, F.Cu at (5.62, -312.4)
- added D18: 1N4148W, Diode_SMD:D_SOD-123, B.Cu at (55.7, -246.8)
- added D19: 1N4148W, Diode_SMD:D_SOD-123, F.Cu at (5.62, -302.3)
- added D20: 1N4148W, Diode_SMD:D_SOD-123, F.Cu at (5.62, -309.0)
- added D21: 1N4148W, Diode_SMD:D_SOD-123, F.Cu at (5.62, -305.7)
- added D22: 1N4148W, Diode_SMD:D_SOD-123, B.Cu at (125.7, -181.1)
- added D23: 1N4148W, Diode_SMD:D_SOD-123, B.Cu at (125.7, -184.5)
- added D24: 1N4148W, Diode_SMD:D_SOD-123, F.Cu at (11.4, -309.0)
- added D25: 1N4148W, Diode_SMD:D_SOD-123, B.Cu at (131.5, -181.1)
- added D26: 1N4148W, Diode_SMD:D_SOD-123, B.Cu at (154.5, -181.1)
- added D27: 1N4148W, Diode_SMD:D_SOD-123, F.Cu at (11.4, -305.7)
- added D28: 1N4148W, Diode_SMD:D_SOD-123, F.Cu at (11.4, -312.4)
- added D29: 1N4148W, Diode_SMD:D_SOD-123, B.Cu at (131.5, -184.5)
- added D3: 1N4148W, Diode_SMD:D_SOD-123, B.Cu at (148.7, -184.5)
- added D30: 1N4148W, Diode_SMD:D_SOD-123, F.Cu at (11.4, -302.3)
- added D31: 1N4148W, Diode_SMD:D_SOD-123, B.Cu at (143.0, -181.1)
- added D32: 1N4148W, Diode_SMD:D_SOD-123, B.Cu at (137.2, -184.5)
- added D33: 1N4148W, Diode_SMD:D_SOD-123, B.Cu at (143.0, -184.5)
- added D34: 1N4148W, Diode_SMD:D_SOD-123, B.Cu at (148.7, -181.1)
- added D35: 1N4148W, Diode_SMD:D_SOD-123, B.Cu at (137.2, -181.1)
- added D36: 1N4148W, Diode_SMD:D_SOD-123, F.Cu at (17.6, -322.5)
- added D37: 1N4148W, Diode_SMD:D_SOD-123, B.Cu at (158.6, -296.0)
- added D38: 1N4148W, Diode_SMD:D_SOD-123, B.Cu at (152.9, -296.0)
- added D39: 1N4148W, Diode_SMD:D_SOD-123, B.Cu at (158.6, -292.7)
- added D4: 1N4148W, Diode_SMD:D_SOD-123, F.Cu at (11.4, -315.7)
- added D40: 1N4148W, Diode_SMD:D_SOD-123, B.Cu at (152.9, -292.7)
- added D41: 1N4148W, Diode_SMD:D_SOD-123, B.Cu at (158.6, -289.3)
- added D42: 1N4148W, Diode_SMD:D_SOD-123, B.Cu at (152.9, -289.3)
- added D43: 1N4148W, Diode_SMD:D_SOD-123, B.Cu at (166.0, -238.9)
- added D44: 1N4148W, Diode_SMD:D_SOD-123, B.Cu at (166.0, -235.6)
- added D45: 1N4148W, Diode_SMD:D_SOD-123, B.Cu at (152.7, -299.4)
- added D46: 1N4148W, Diode_SMD:D_SOD-123, B.Cu at (166.0, -228.9)
- added D47: 1N4148W, Diode_SMD:D_SOD-123, B.Cu at (166.0, -184.5)
- added D48: 1N4148W, Diode_SMD:D_SOD-123, B.Cu at (166.0, -181.1)
- added D49: 1N4148W, Diode_SMD:D_SOD-123, B.Cu at (160.2, -184.5)
- added D5: 1N4148W, Diode_SMD:D_SOD-123, F.Cu at (17.6, -329.2)
- added D50: 1N4148W, Diode_SMD:D_SOD-123, B.Cu at (160.2, -181.1)
- added D51: 1N4148W, Diode_SMD:D_SOD-123, B.Cu at (154.5, -184.5)
- added D52: 1N4148W, Diode_SMD:D_SOD-123, B.Cu at (196.9, -267.3)
- added D53: 1N4148W, Diode_SMD:D_SOD-123, B.Cu at (196.9, -277.3)
- added D54: 1N4148W, Diode_SMD:D_SOD-123, B.Cu at (191.1, -277.3)
- added D55: 1N4148W, Diode_SMD:D_SOD-123, B.Cu at (202.6, -274.0)
- added D56: 1N4148W, Diode_SMD:D_SOD-123, B.Cu at (196.9, -274.0)
- added D57: 1N4148W, Diode_SMD:D_SOD-123, B.Cu at (191.1, -274.0)
- added D58: 1N4148W, Diode_SMD:D_SOD-123, B.Cu at (202.6, -270.6)
- added D59: 1N4148W, Diode_SMD:D_SOD-123, B.Cu at (196.9, -270.6)
- added D6: 1N4148W, Diode_SMD:D_SOD-123, F.Cu at (17.6, -325.8)
- added D60: 1N4148W, Diode_SMD:D_SOD-123, B.Cu at (202.6, -267.3)
- added D61: 1N4148W, Diode_SMD:D_SOD-123, B.Cu at (202.6, -277.3)
- added D62: 1N4148W, Diode_SMD:D_SOD-123, B.Cu at (202.6, -263.9)
- added D63: 1N4148W, Diode_SMD:D_SOD-123, B.Cu at (196.9, -263.9)
- added D64: 1N4148W, Diode_SMD:D_SOD-123, B.Cu at (191.1, -270.6)
- added D65: 1N4148W, Diode_SMD:D_SOD-123, B.Cu at (191.1, -267.3)
- added D66: 1N4148W, Diode_SMD:D_SOD-123, B.Cu at (191.1, -263.9)
- added D67: 1N4148W, Diode_SMD:D_SOD-123, B.Cu at (202.6, -260.6)
- added D68: 1N4148W, Diode_SMD:D_SOD-123, B.Cu at (166.0, -232.2)
- added D7: 1N4148W, Diode_SMD:D_SOD-123, F.Cu at (11.8, -322.5)
- added D8: 1N4148W, Diode_SMD:D_SOD-123, B.Cu at (55.7, -243.5)
- added D9: 1N4148W, Diode_SMD:D_SOD-123, B.Cu at (49.9, -246.8)
- added R2: 10k, Resistor_SMD:R_1206_3216Metric_Pad1.42x1.75mm_HandSolder, B.Cu at (158.5, -299.4)
- added SW10: 9, acheron_MX:MX100, B.Cu at (-238.1, -347.7)
- added SW11: 0, acheron_MX:MX100, B.Cu at (-219.1, -347.7)
- added SW12: _, acheron_MX:MX100, B.Cu at (-200.0, -347.7)
- added SW13: =/+, acheron_MX:MX100, B.Cu at (-181.0, -347.7)
- added SW14: Backspace_200, acheron_MX:MX200, B.Cu at (-152.4, -347.7)
- added SW15: M1, acheron_MX:MX100, B.Cu at (-123.8, -347.7)
- added SW16: Tab_150, acheron_MX:MX150, B.Cu at (-404.8, -328.6)
- added SW17: Q, acheron_MX:MX100, B.Cu at (-381.0, -328.6)
- added SW18: W, acheron_MX:MX100, B.Cu at (-361.9, -328.6)
- added SW19: E, acheron_MX:MX100, B.Cu at (-342.9, -328.6)
- added SW20: R, acheron_MX:MX100, B.Cu at (199.1, -228.6)
- added SW21: T, acheron_MX:MX100, B.Cu at (108.9, -236.5)
- added SW22: Y, acheron_MX:MX100, B.Cu at (70.8, -278.7)
- added SW23: U, acheron_MX:MX100, B.Cu at (34.9, -319.0)
- added SW24: I, acheron_MX:MX100, B.Cu at (158.8, -196.2)
- added SW25: O, acheron_MX:MX100, B.Cu at (138.6, -216.4)
- added SW26: P, acheron_MX:MX100, B.Cu at (178.9, -210.4)
- added SW27: {, acheron_MX:MX100, B.Cu at (108.9, -256.7)
- added SW28: }, acheron_MX:MX100, B.Cu at (88.8, -256.7)
- added SW29: \, acheron_MX:MX100, B.Cu at (91.0, -276.8)
- added SW3: 2, acheron_MX:MX100, B.Cu at (-371.5, -347.7)
- added SW30: M2, acheron_MX:MX100, B.Cu at (178.9, -190.2)
- added SW31: Caps, acheron_MX:MX175, B.Cu at (252.4, -268.9)
- added SW32: A, acheron_MX:MX100, B.Cu at (158.8, -216.4)
- added SW33: S, acheron_MX:MX100, B.Cu at (55.1, -319.0)
- added SW34: D, acheron_MX:MX100, B.Cu at (84.8, -298.9)
- added SW35: F, acheron_MX:MX100, B.Cu at (199.1, -188.3)
- added SW36: G, acheron_MX:MX100, B.Cu at (30.5, -278.7)
- added SW37: H, acheron_MX:MX100, B.Cu at (149.2, -236.5)
- added SW38: J, acheron_MX:MX100, B.Cu at (129.1, -256.7)
- added SW39: K, acheron_MX:MX100, B.Cu at (111.1, -276.8)
- added SW4: 3, acheron_MX:MX100, F.Cu at (-352.4, -347.7)
- added SW40: L, acheron_MX:MX100, B.Cu at (75.2, -319.0)
- added SW41: :, acheron_MX:MX100, B.Cu at (149.2, -256.7)
- added SW42: ", acheron_MX:MX100, B.Cu at (131.3, -276.8)
- added SW43: Enter_2.25, acheron_MX:MX225, B.Cu at (247.6, -291.0)
- added SW44: M3, acheron_MX:MX100, B.Cu at (169.4, -250.7)
- added SW45: LShift_225, acheron_MX:MX225, B.Cu at (127.4, -319.0)
- added SW46: x, acheron_MX:MX100, B.Cu at (178.9, -230.5)
- added SW47: x, acheron_MX:MX100, B.Cu at (199.1, -208.5)
- added SW48: c, acheron_MX:MX100, B.Cu at (219.2, -188.3)
- added SW49: v, acheron_MX:MX100, B.Cu at (104.9, -297.0)
- added SW5: 4, acheron_MX:MX100, B.Cu at (-333.4, -347.7)
- added SW50: b, acheron_MX:MX100, B.Cu at (239.4, -188.3)
- added SW51: n, acheron_MX:MX100, B.Cu at (219.2, -208.5)
- added SW52: m, acheron_MX:MX100, B.Cu at (209.7, -248.8)
- added SW53: <, acheron_MX:MX100, B.Cu at (44.5, -298.9)
- added SW54: >, acheron_MX:MX100, B.Cu at (259.5, -208.5)
- added SW55: ?, acheron_MX:MX100, B.Cu at (239.4, -228.6)
- added SW56: R-shift_175, acheron_MX:MX175, B.Cu at (132.2, -297.0)
- added SW57: UP, acheron_MX:MX100, B.Cu at (95.4, -319.0)
- added SW58: M4, acheron_MX:MX100, B.Cu at (259.5, -228.6)
- added SW59: LCTRL, acheron_MX:MX125, B.Cu at (232.2, -248.8)
- added SW6: 5, acheron_MX:MX100, B.Cu at (-314.3, -347.7)
- added SW60: Win, acheron_MX:MX125, B.Cu at (174.0, -291.0)
- added SW61: Alt, acheron_MX:MX125, B.Cu at (257.1, -248.8)
- added SW62: Space, acheron_MX:MX625R, B.Cu at (209.5, -317.4)
- added SW63: Alt, acheron_MX:MX100, B.Cu at (259.5, -188.3)
- added SW64: Win, acheron_MX:MX100, B.Cu at (219.2, -228.6)
- added SW65: Menu, acheron_MX:MX100, B.Cu at (176.3, -270.8)
- added SW66: LEFT, acheron_MX:MX100, B.Cu at (151.4, -276.8)
- added SW67: DOWN, acheron_MX:MX100, B.Cu at (189.5, -250.7)
- added SW68: RIGHT, acheron_MX:MX100, B.Cu at (239.4, -208.5)
- added SW7: 6, acheron_MX:MX100, B.Cu at (-295.3, -347.7)
- added SW8: 7, acheron_MX:MX100, B.Cu at (-276.2, -347.7)
- added SW9: 8, acheron_MX:MX100, B.Cu at (-257.2, -347.7)
- C1: renamed from C5; moved to B.Cu
- C2: renamed from C6; moved to B.Cu
- C3: renamed from C7; moved to B.Cu
- C4: renamed from C8; moved to B.Cu
- C5: renamed from C1; moved to B.Cu
- C6: renamed from C2; moved to B.Cu
- C7: renamed from C3; moved to B.Cu
- C8: renamed from C4; moved to B.Cu
- D1: value D_Small -> 1N4148W; moved to B.Cu
- D2: renamed from D3; value D_Small -> 1N4148W; moved to B.Cu
- D2, D4, J1, R1, R3, R4, SWP1, U1, Y1: moved to B.Cu
- R1: renamed from R2; moved to B.Cu
- R5: value 10k -> 1k; moved to B.Cu
- SW1: renamed from SW2; value MXSwitch -> tilde/esc
- SW2: renamed from SW4; value MXSwitch -> 1
- moved SW1 560.2 mm to (-409.6, -347.7)
- moved SW2 529.2 mm to (-390.5, -347.7)
- moved C6 71.9 mm to (-1.35, -46.7), turned to 180 degrees
- moved C7 68.5 mm to (19.1, -70.5)
- moved R5 67.2 mm to (8.54, -62.1)
- moved C1 67.1 mm to (13.9, -61.9)
- moved C4 65.8 mm to (19.1, -67.6)
- moved C2 65.0 mm to (-17.3, -28.8)
- moved C8 65.0 mm to (-6.51, -37.2)
- moved D4 65.0 mm to (-22.5, -28.6)
- moved J1 65.0 mm to (11.1, -67.7)
- moved R1 65.0 mm to (-40.3, -28.6)
- moved R1 65.0 mm to (-46.2, -28.6)
- moved R3 65.0 mm to (-34.3, -28.6)
- moved R4 65.0 mm to (-28.4, -28.6)
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Connections:
- C5 pad 1: GND -> Net-(C5-Pad1)
- D1 pad 1: Col1 -> Row1
- D2 pad 1: Col1 -> Row1
- D2 pad 2: Net-(D3-Pad2) -> Net-(D2-Pad2)
- SW2 pad 1: Col1 -> Col2
- SW2 pad 2: Net-(D3-Pad2) -> Net-(D2-Pad2)
- SWP1 pad 1: GND -> Net-(C5-Pad1)
- SWP1 pad 2: Net-(R1-Pad2) -> RST

Commit message: grind done
Parts:
- removed the SW3 at (-19.0, -60.5)
- removed the SW5 at (-39.1, -60.5)
- SW29: footprint acheron_MX:MX100 -> acheron_MX:MX150
- SW46: value x -> z
- moved SW31 656.1 mm to (-402.4, -309.6)
- moved SW59 639.8 mm to (-407.2, -271.5)
- moved SW61 617.1 mm to (-359.6, -271.5)
- moved SW60 557.7 mm to (-383.4, -271.5)
- moved SW48 557.3 mm to (-328.6, -290.5)
- moved SW47 552.8 mm to (-347.7, -290.5)
- moved SW46 548.9 mm to (-366.7, -290.5)
- moved SW32 543.0 mm to (-376.2, -309.6)
- moved SW50 539.6 mm to (-290.5, -290.5)
- moved SW20 532.4 mm to (-323.9, -328.6)
- moved SW35 532.1 mm to (-319.1, -309.6)
- moved SW45 525.9 mm to (-397.7, -290.5)
- moved SW62 499.7 mm to (-288.1, -271.5)
- moved SW51 497.5 mm to (-271.5, -290.5)
- moved SW63 485.7 mm to (-219.1, -271.5)
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
Commit message: ep 3 end
Parts:
- removed J1: USB_B_Mini, acheron_Connectors:USB_MiniB_XM7D-0512
- added Je: USB_B_Mini, acheron_Connectors:USB_MiniB_XM7D-0512, B.Cu at (-400.1, -353.2)
- SW4: moved to B.Cu
- turned SW4 to 180 degrees
Other:
- board outline added: 309.6 x 100 mm

Commit message: pp
Parts:
- SW1, SW2: moved to B.Cu
- turned SW1 to 180 degrees
- turned SW2 to 180 degrees

Commit message: connecto
Parts:
- removed the D2 at (19.6, -64.4)
- removed the D4 at (-22.5, -28.6)
- removed the R1 at (-46.2, -28.6)
- D1, D11, D12, D13, D14, D15, D16, D18, D2, D22, D23, D25, D26, D29, D3, D31, D32, D33, D34, D35, D37, D38, D39, D40, D41, D42, D43, D44, D45, D46, D47, D48, D49, D50, D51, D52, D53, D54, D55, D56, D57, D58, D59, D60, D61, D62, D63, D64, D65, D66, D67, D68, D8, D9: footprint Diode_SMD:D_SOD-123 -> acheron_Components:D_THT_7.62mm_SOD-123
- D10, D17, D19, D20, D21, D24, D27, D28, D30, D36, D4, D5, D6, D7: footprint Diode_SMD:D_SOD-123 -> acheron_Components:D_THT_7.62mm_SOD-123; moved to B.Cu
- R2: value 10k -> 330
- moved D59 604.1 mm to (-407.2, -266.7)
- moved D60 586.0 mm to (-383.4, -266.7)
- moved D61 562.3 mm to (-359.6, -266.7)
- moved D31 559.2 mm to (-402.4, -304.8)
- moved D45 550.5 mm to (-397.7, -285.8)
- moved D3 543.8 mm to (-371.5, -342.9)
- moved D16 543.0 mm to (-404.8, -323.9)
- moved D46 535.7 mm to (-366.7, -285.8)
- moved D32 527.4 mm to (-376.2, -304.8)
- moved D47 523.5 mm to (-347.7, -285.8)
- moved D33 514.4 mm to (-357.2, -304.8)
- moved D1 510.9 mm to (-409.6, -342.9)
- moved D2 507.0 mm to (-390.5, -342.9)
- moved D48 505.5 mm to (-328.6, -285.8)
- moved D34 502.3 mm to (-338.1, -304.8)
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- renumbered Je to J1
Connections:
- C5 pad 1: Net-(C5-Pad1) -> GND
- D66 pad 1: Net-(D66-Pad1) -> Row5
- R2 pad 2: Net-(C5-Pad1) -> Net-(R2-Pad2)
- SWP1 pad 1: Net-(C5-Pad1) -> Net-(R2-Pad2)
- U1 pad 10: Net-(U1-Pad10) -> Col3
- U1 pad 11: Net-(U1-Pad11) -> Col4
- U1 pad 12: Net-(U1-Pad12) -> Col8
- U1 pad 18: Net-(U1-Pad18) -> Col11
- U1 pad 19: Net-(U1-Pad19) -> Col12
- U1 pad 20: Net-(U1-Pad20) -> Col13
- U1 pad 21: Net-(U1-Pad21) -> Col14
- U1 pad 22: Net-(U1-Pad22) -> Row1
- U1 pad 25: Net-(U1-Pad25) -> Col15
- U1 pad 26: Net-(U1-Pad26) -> Row2
- U1 pad 27: Net-(U1-Pad27) -> Col15
- U1 pad 28: Net-(U1-Pad28) -> Col5
- U1 pad 29: Net-(U1-Pad29) -> Col6
- U1 pad 30: Net-(U1-Pad30) -> Col7
- U1 pad 31: Net-(U1-Pad31) -> Col9
- U1 pad 32: Net-(U1-Pad32) -> Col10
- U1 pad 8: Net-(U1-Pad8) -> Col1
- U1 pad 9: Net-(U1-Pad9) -> Col2

Commit message: onboard mcu
Parts:
- D1, D10, D11, D12, D13, D14, D15, D16, D17, D18, D19, D2, D20, D21, D22, D23, D24, D25, D26, D27, D28, D29, D3, D30, D31, D32, D33, D34, D35, D36, D37, D38, D39, D4, D40, D41, D42, D43, D44, D45, D46, D47, D48, D49, D5, D50, D51, D52, D53, D54, D55, D56, D57, D58, D59, D6, D60, D61, D62, D63, D64, D65, D66, D67, D68, D7, D8, D9: footprint acheron_Components:D_THT_7.62mm_SOD-123 -> acheron_Components:D_SOD-123
- moved R2 393.7 mm to (-297.7, -261.9)
- moved SWP1 392.6 mm to (-304.8, -273.8)
- moved Y1 365.3 mm to (-269.3, -281.0), turned to 0 degrees
- moved C7 362.6 mm to (-276.2, -281.0), turned to 270 degrees
- moved C8 351.9 mm to (-277.2, -261.9)
- moved C6 350.4 mm to (-261.9, -281.0), turned to 270 degrees
- moved C3 349.0 mm to (-247.7, -264.3), turned to 270 degrees
- moved R4 345.4 mm to (-278.6, -266.7), turned to 90 degrees
- moved R3 344.5 mm to (-283.4, -266.7), turned to 90 degrees
- moved C1 338.3 mm to (-257.2, -264.3), turned to 270 degrees
- moved C5 337.6 mm to (-244.2, -276.2)
- moved C4 335.3 mm to (-252.4, -264.3), turned to 270 degrees
- moved R5 326.8 mm to (-244.4, -269.1), turned to 180 degrees
- moved C2 326.1 mm to (-242.9, -264.3), turned to 270 degrees
- moved R1 321.8 mm to (-247.7, -274.7), turned to 90 degrees
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
Commit message: final prior to test routing
Parts:
- moved C6 147.9 mm to (-404.8, -319.1)
- moved C7 147.9 mm to (-419.1, -319.1)
- moved Y1 147.9 mm to (-412.2, -319.1)
- moved C5 146.6 mm to (-387.0, -309.6), turned to 270 degrees
- moved R1 140.7 mm to (-384.6, -307.2)
- moved R3 140.1 mm to (-402.4, -340.5)
- moved R4 140.1 mm to (-397.7, -340.5)
- moved R5 138.8 mm to (-373.9, -319.1), turned to 270 degrees
- moved C2 133.2 mm to (-364.3, -319.1)
- moved U1 132.7 mm to (-390.5, -319.1), turned to 90 degrees
- moved C3 131.1 mm to (-366.7, -319.1)
- moved C4 128.9 mm to (-369.1, -319.1)
- moved C1 126.7 mm to (-371.5, -319.1)
- moved C8 123.4 mm to (-390.5, -310.9)
- moved R2 108.2 mm to (-397.7, -303.3), turned to 270 degrees
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
Commit message: diode switch
Parts:
- moved D19 4.29 mm to (-346.5, -321.5), turned to 90 degrees
- moved D23 4.29 mm to (-270.3, -321.5), turned to 90 degrees
- moved D31 4.29 mm to (-406.0, -302.4), turned to 90 degrees
- moved D34 4.29 mm to (-341.7, -302.4), turned to 90 degrees
- moved D35 4.29 mm to (-322.7, -302.4), turned to 90 degrees
- moved D45 4.29 mm to (-401.2, -283.4), turned to 90 degrees
- moved D46 4.29 mm to (-370.3, -283.4), turned to 90 degrees
- moved D50 4.29 mm to (-294.1, -283.4), turned to 90 degrees
- moved D51 4.29 mm to (-275.0, -283.4), turned to 90 degrees
- moved D24 4.29 mm to (-251.2, -321.5), turned to 90 degrees
- moved D25 4.29 mm to (-232.2, -321.5), turned to 90 degrees
- moved D27 4.29 mm to (-194.1, -321.5), turned to 90 degrees
- moved D28 4.29 mm to (-175.0, -321.5), turned to 90 degrees
- moved D29 4.29 mm to (-151.2, -321.5), turned to 90 degrees
- moved D39 4.29 mm to (-246.5, -302.4), turned to 90 degrees
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Routing:
- net GND: track 0.00 -> 116.5 mm
- net Net-(R3-Pad1): track 0.00 -> 38.5 mm, vias 0 -> 2
- net Net-(R4-Pad1): track 0.00 -> 34.7 mm, vias 0 -> 2
- net +5V: track 0.00 -> 22.1 mm
- net Net-(R5-Pad2): track 0.00 -> 20.2 mm, vias 0 -> 2
- net RST: track 0.00 -> 19.1 mm
- net Net-(J1-Pad2): track 0.00 -> 14.5 mm
- net Net-(C6-Pad1): track 0.00 -> 14.2 mm
- net Net-(J1-Pad3): track 0.00 -> 11.0 mm, vias 0 -> 1
- net Net-(C7-Pad1): track 0.00 -> 4.75 mm
- net Net-(R2-Pad2): track 0.00 -> 4.51 mm
- net Net-(C8-Pad1): track 0.00 -> 2.89 mm
