File: mrkeebstutorial.kicad_pcb (KiCad board)
At the start: 2 copper layers, 309.6 x 100 mm, 153 parts, among them J1 USB_B_Mini, SW1 tilde/esc, SW10 9, SW11 0, SW12 _, SW13 =/+, SW14 Backspace_200, SW15 M1, SW16 Tab_150, SW17 Q, SW18 W, SW19 E, SW2 1, SW20 R, SW21 T, SW22 Y, SW23 U, SW24 I, SW25 O, SW26 P, SW27 {, SW28 }, SW29 \, SW3 2, SW30 M2, SW31 Caps, SW32 A, SW33 S, SW34 D, SW35 F, SW36 G, SW37 H, SW38 J, SW39 K, SW4 3, SW40 L, SW41 :, SW42 ", SW43 Enter_2.25, SW44 M3, SW45 LShift_225, SW46 z, SW47 x, SW48 c, SW49 v, SW5 4, SW50 b, SW51 n, SW52 m, SW53 <, SW54 >, SW55 ?, SW56 R-shift_175, SW57 UP, SW58 M4, SW59 LCTRL, SW6 5, SW60 Win, SW61 Alt, SW62 Space, SW63 Alt, SW64 Win, SW65 Menu, SW66 LEFT, SW67 DOWN, SW68 RIGHT, SW7 6, SW8 7, SW9 8, U1 ATmega32U4-AU, Y1 16MHz

Commit message: changed ground plane
Parts:
- moved SW31 0.07 mm to (-402.5, -309.5)
Connections:
- U1 pad 10: Col3 -> Col4
- U1 pad 11: Col4 -> Net-(U1-Pad11)
- U1 pad 13: Net-(U1-Pad13) -> RST
- U1 pad 20: Net-(U1-Pad20) -> Col1
- U1 pad 21: Col1 -> Row1
- U1 pad 22: Row1 -> Row2
- U1 pad 37: RST -> Net-(U1-Pad37)
- U1 pad 8: Row2 -> Col2
- U1 pad 9: Col2 -> Col3
Routing:
- net GND: track 117.2 -> 60.9 mm, vias 5 -> 8
- net Row2: track 331.8 -> 312.2 mm, vias 7 -> 2
- net RST: track 36.5 -> 50.4 mm, vias 0 -> 2
- net Row1: track 330.6 -> 324.8 mm, vias 2 -> 1
- net Net-(R4-Pad1): track 34.3 -> 31.2 mm
- net +5V: track 128.7 -> 126.8 mm
- net Col4: track 139.2 -> 140.7 mm
- net Row3: track 301.5 -> 302.7 mm
- net Col2: track 124.1 -> 123.1 mm
- net Net-(U1-Pad11): track 0.00 -> 0.73 mm
- net Col3: track 144.3 -> 143.7 mm
- net Col1: track 90.0 -> 90.5 mm
- added copper zone on F.Cu, net GND
- removed copper zone on B.Cu, net GND

Commit message: migraterd dshit
Routing:
- net Col7: track 179.8 -> 199.9 mm
- net Col2: track 123.1 -> 123.9 mm
